Commit message: Add rviz_example dynamic_joint_states

File: src/rviz_example/base_world_bringup/urdf/basic_world.urdf (robot description, URDF)
Before this commit: robot base_world, 3 links, 2 joints
Links:
- added link dynamic_joint_frame_link
- added link extension_joint_frame_link
Joints:
- added joint dynamic_joint_conti: type continuous, parent base_frame_link, child dynamic_joint_frame_link, origin xyz=0.5 0.5 0.5 rpy=0 0 0, axis 0 0 1
- added joint extension_joint_fixed: type fixed, parent dynamic_joint_frame_link, child extension_joint_frame_link, origin xyz=1 1 1 rpy=0 0 0
- joint base_joint_fixed: origin xyz=1 1 1 rpy=0 0 0 -> xyz=1 1 0 rpy=0 0 0
